File: Kicad/CO2Dot.kicad_sch (KiCad schematic)
At the start: 20 parts, among them J1 Conn_01x08, J3 Conn_01x02_Socket, U1 AS7341/3, U4 BME680, U5 AP7312-1833W6-7, U8 ESP8685, Y2 40MHz

Commit message: PCB CO2Dot with BME, V002 (squashed)
Parts:
- removed J3: Conn_01x02_Socket, Connector_PinHeader_2.54mm:PinHeader_1x02_P2.54mm_Vertical, symbol Connector:Conn_01x02_Socket
- removed U4: BME680, Package_LGA:Bosch_LGA-8_3x3mm_P0.8mm_ClockwisePinNumbering, symbol Sensor:BME680
- added C1, C4: 2.2u, Capacitor_SMD:C_0603_1608Metric_Pad1.08x0.95mm_HandSolder, symbol Device:C
- added C6: 10u, Capacitor_SMD:C_0603_1608Metric, symbol Device:C
- added D1: 1N4148WT, Diode_SMD:D_SOD-123, symbol Diode:1N4148WT
- added D3: LED, Diode_SMD:D_0805_2012Metric, symbol Device:LED
- added J2: USB_C_Receptacle, Connector_USB:USB_C_Receptacle_HRO_TYPE-C-31-M-12, symbol Connector:USB_C_Receptacle
- added J4: Conn_01x02_Pin, Connector_PinHeader_2.54mm:PinHeader_1x02_P2.54mm_Vertical, symbol Connector:Conn_01x02_Pin
- added J5: secondBoard, Connector_PinSocket_1.27mm:PinSocket_1x04_P1.27mm_Vertical, symbol Connector:Conn_01x04_Pin
- added R10, R11: 0, Resistor_SMD:R_0603_1608Metric_Pad0.98x0.95mm_HandSolder, symbol Device:R
- added R12, R13, R29, R30: 5.1K, Resistor_SMD:R_0603_1608Metric, symbol main-rescue:R-
- added R7, R8: 10K, Resistor_SMD:R_0603_1608Metric_Pad0.98x0.95mm_HandSolder, symbol Device:R
- added R9: 500, Resistor_SMD:R_0603_1608Metric_Pad0.98x0.95mm_HandSolder, symbol Device:R
- added SW2: SW_Push, Button_Switch_SMD:SW_SPST_EVQP2_ShortPushTravel_H2.1mm, symbol Switch:SW_Push
- added U2: IP4234CZ6, Package_TO_SOT_SMD:SC-74-6_1.55x2.9mm_P0.95mm, symbol Power_Protection:IP4234CZ6
- added U3: BME688, Personal_Library:BME688, symbol Personal_Library:BME688
- C10, C11, C3: MANUFACTURER CL05A225MQ5NNNC -> (none); Manufacturer_Part_Number (none) -> GRT188R61H225KE13D
- C12: Manufacturer_Part_Number (none) -> GRT188R61H225KE13D
- C2, C9: value 100n -> 2.2u; MANUFACTURER CL05A225MQ5NNNC -> (none); Manufacturer_Part_Number (none) -> GRT188R61H225KE13D
- D2: footprint Personal_Library:NF2W757GT-F1 -> Diode_SMD:D_0805_2012Metric; now not fitted; now left out of the parts list
- J1, R1: now not fitted; now left out of the parts list
- R2: value 10K -> 5.1K; footprint Resistor_SMD:R_0603_1608Metric_Pad0.98x0.95mm_HandSolder -> Resistor_SMD:R_0603_1608Metric; Manufacturer_Part_Number (none) -> 652-CR0603FX-5101ELF
- R3: value 10K -> 0R; now not fitted; now left out of the parts list
- R4, R5: now not fitted
- R6: value 12K -> 0R; now not fitted; now left out of the parts list
- U1: value AS7341/3 -> AS7341-DLGT; footprint Personal_Library:XDCR_AS7341-DLGM -> PSON80P310X200X110-8N; Manufacturer_Part_Number (none) -> AS7341-DLGM
- U5: footprint Package_TO_SOT_SMD:TSOT-23-6_HandSoldering -> Package_TO_SOT_SMD:TSOT-23-6; Manufacturer_Part_Number (none) -> AP7312-1833W6-7
- U8: Manufacturer_Part_Number (none) -> ESP8685H4
- Y2: Manufacturer_Part_Number (none) -> ECS-400-8-47B2-CKM-TR
Connections:
- net BOOT: now also R12.1, SW2.1
- net GND: now also C1.2, C4.2, C6.1, J2.A1 (GND), J2.A12 (GND), J2.B1 (GND), J2.B12 (GND), J2.S1 (SHIELD), J5.1 (Pin_1), R13.1, R29.1, R30.1, SW2.2, U2.2 (VN), U3.1 (GND), U3.5 (SDO), U3.7 (GND__1); no longer R6.1
- net LED1ACT: now also J4.2 (Pin_2), R10.2, R11.2
- net Rxd: now also R11.1, R9.2; no longer U8.23 (U0RXD/GPIO20)
- net SCL: now also R3.2, R8.1, U3.4 (SCK)
- net SDA: now also R6.2, R7.1, U3.3 (SDI)
- net Txd: now also R10.1
- net V+: now also C1.1, D1.1 (K), J4.1 (Pin_1)
- net V+1.8V: now also C4.1, J5.2 (Pin_2)
- net V+3V: now also R12.2, R7.2, R8.2, U3.2 (CSB), U3.6 (VDDIO), U3.8 (VDD)
- net at U8.13 (MTDO/GPIO7): no longer R3.1
- net D-: now reaches U8.21 (GPIO18/USB_D-)
- net D-: now also U2.4
- net D+: now reaches U8.22 (GPIO19/USB_D+)
- net D+: now also U2.3
- net SDA_2: now reaches U8.4 (GPIO0/XTAL_32K_P/ADC1_CH0)
- net SDA_2: now also R3.1, J5.3 (Pin_3)
- net SCL_2: now reaches U8.5 (GPIO1/XTAL_32K_N/ADC1_CH1)
- net SCL_2: now also R6.1, J5.4 (Pin_4)
- net GPIO-ADPD: no longer names the net of U8.16 (GPIO10)
- net GPIO-ADPD: now also D3.2 (A)
- removed net SYNC: R3.2, R6.2, U1.6 (GPIO)
- new net: D3.1 (K), R13.2
- new net: R9.1, U8.23 (U0RXD/GPIO20)
- new net: J2.A6 (D+), J2.B6 (D+), U2.1
- new net: J2.A7 (D-), J2.B7 (D-), U2.6
- new net CC1: J2.A5 (CC1), R29.2
- new net CC2: J2.B5 (CC2), R30.2
- new net Vusb: C6.2, D1.2 (A), J2.A4 (VBUS), J2.A9 (VBUS), J2.B4 (VBUS), J2.B9 (VBUS), U2.5 (VP)
- no-connect marks 8 -> 16
Other:
- note added: "Changes 1.0 - 1.1 * 1N4148 package * new status LED - D3 * button footprint change"
- note removed: "BOOT&RESET"
- note removed: "Constant current FLSH"
- note removed: "On top"
- moved on the sheet: C10, C11, C12, C2, C3, C9, R2, U1, U5, U8, Y2
