File: Kicad/CO2Dot.kicad_pcb (KiCad board)
At the start: 4 copper layers, 25 x 40 mm, 31 parts, among them J2 USB_C_Receptacle, J4 Conn_01x02_Pin, J5 secondBoard, SW2 SW_Push, U1 AS7341-DLGT, U2 IP4234CZ6, U3 BME688, U5 AP7312-1833W6-7, U8 ESP8685, Y2 40MHz

Commit message: (kicad) fixed unconnected
Routing:
- net V+3V: track 37.0 -> 37.8 mm

Commit message: (kicad) board rev 0.0.1
Routing:
- net V+: vias 5 -> 6
- net GND: vias 34 -> 33
Changed lines of the file:
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@@
-	)
-	(via
-		(at 95.206024 110.011064)
-		(size 0.6)
-		(drill 0.3)
-		(layers "F.Cu" "B.Cu")
-		(capping no)
-		(covering
-			(front no)
-			(back no)
-		)
-		(plugging
-			(front no)
-			(back no)
-		)
-		(filling no)
-		(net "GND")
 	)
 	(via
@@
 		(size 0.6)
 		(drill 0.3)
+		(layers "F.Cu" "B.Cu")
+		(capping no)
+		(covering
+			(front no)
+			(back no)
+		)
+		(plugging
+			(front no)
+			(back no)
+		)
+		(filling no)
+		(net "V+")
+	)
+	(via
+		(at 94.5 110)
+		(size 0.6)
+		(drill 0.3)

Commit message: (kicad-freeCAD) CO2 v0.0.3
Parts:
- removed J5: secondBoard, Connector_PinSocket_1.27mm:PinSocket_1x04_P1.27mm_Vertical
- moved U1 7.45 mm to (103.3, 107.9)
- moved U3 7.23 mm to (95.2, 107.6)
- moved D2 7.11 mm to (103.3, 104.7)
- moved C9 5.49 mm to (100.8, 107.1), turned to 90 degrees
Routing:
- net V+3V: track 37.8 -> 60.2 mm
- net SCL_2: track 23.3 -> 2.75 mm, vias 1 -> 0
- net SDA_2: track 29.4 -> 12.6 mm, vias 1 -> 0
- net V+1.8V: track 38.2 -> 28.7 mm, vias 0 -> 2
- net LED1ACT: track 19.6 -> 27.2 mm
- net SDA: track 34.6 -> 40.8 mm
- net SCL: track 35.2 -> 40.1 mm
- net V+: track 32.4 -> 28.6 mm, vias 6 -> 2
- net GND: track 34.9 -> 35.4 mm, vias 33 -> 28
Other:
- outline, holes or cut-outs redrawn
- board text added: "CO2Dot V0.0.3"
- board text removed: "CO2Dot V0.02 LG/LC"
